Commit message: add the cover link

File: rosbot_description/urdf/rosbot.urdf.xacro (robot description, xacro)
@@ -7,5 +7,5 @@
                 <mesh filename="package://rosbot_description/meshes/rosbot/body.stl" scale="0.001 0.001 0.001"/>
             </geometry>
-            <origin xyz="0 0 0" rpy="0 0 0"/>
+            <origin xyz="0 0 0" rpy="${pi/2} 0 ${pi/2}"/>
         </visual>
     </link>
@@ -15,3 +15,16 @@
         <origin xyz="0 0 0" rpy="0 0 0"/>
     </joint>
+    <link name="cover_link">
+        <visual>
+            <geometry>
+                <mesh filename="package://rosbot_description/meshes/rosbot/cover.stl" scale="0.001 0.001 0.001"/>
+            </geometry>
+            <origin xyz="0 0 0.015" rpy="${pi/2} 0 ${pi/2}"/>
+        </visual>
+    </link>
+    <joint name="cover_joint" type="fixed">
+        <parent link="base_link"/>
+        <child link="cover_link"/>
+        <origin xyz="0 0 0.0603" rpy="0 0 0"/>
+    </joint>
 </robot>

Commit message: add the wheel to urdf

File: rosbot_description/urdf/rosbot.urdf.xacro (robot description, xacro)
@@ -1,4 +1,7 @@
 <?xml version="1.0"?>
 <robot name="rosbot" xmlns:xacro="http://ros.org/wiki/xacro">
+    <xacro:property name="wheel_radius" value="0.0425"/>
+    <xacro:property name="wheel_separation_x" value="0.106"/>
+    <xacro:property name="wheel_separation_y" value="0.192"/>
     <link name="base_footprint"/>
     <link name="base_link">
@@ -13,5 +16,5 @@
         <parent link="base_footprint"/>
         <child link="base_link"/>
-        <origin xyz="0 0 0" rpy="0 0 0"/>
+        <origin xyz="0 0 ${wheel_radius}" rpy="0 0 0"/>
     </joint>
     <link name="cover_link">
@@ -28,3 +31,55 @@
         <origin xyz="0 0 0.0603" rpy="0 0 0"/>
     </joint>
+    <link name="wheel_left_back_link">
+        <visual>
+            <geometry>
+                <mesh filename="package://rosbot_description/meshes/rosbot/wheel_a.dae"/>
+            </geometry>
+            <origin xyz="0 0 0" rpy="0 0 0"/>
+        </visual>
+    </link>
+    <joint name="wheel_left_back_joint" type="fixed">
+        <parent link="base_link"/>
+        <child link="wheel_left_back_link"/>
+        <origin xyz="-${wheel_separation_x/2} ${wheel_separation_y/2} 0.015" rpy="0 0 0"/>
+    </joint>
+    <link name="wheel_left_forward_link">
+        <visual>
+            <geometry>
+                <mesh filename="package://rosbot_description/meshes/rosbot/wheel_a.dae"/>
+            </geometry>
+            <origin xyz="0 0 0" rpy="0 0 0"/>
+        </visual>
+    </link>
+    <joint name="wheel_left_forward_joint" type="fixed">
+        <parent link="base_link"/>
+        <child link="wheel_left_forward_link"/>
+        <origin xyz="${wheel_separation_x/2} ${wheel_separation_y/2} 0.015" rpy="0 0 0"/>
+    </joint>
+    <link name="wheel_right_back_link">
+        <visual>
+            <geometry>
+                <mesh filename="package://rosbot_description/meshes/rosbot/wheel_b.dae"/>
+            </geometry>
+            <origin xyz="0 0 0" rpy="0 0 0"/>
+        </visual>
+    </link>
+    <joint name="wheel_right_back_joint" type="fixed">
+        <parent link="base_link"/>
+        <child link="wheel_right_back_link"/>
+        <origin xyz="-${wheel_separation_x/2} -${wheel_separation_y/2} 0.015" rpy="0 0 0"/>
+    </joint>
+    <link name="wheel_right_forward_link">
+        <visual>
+            <geometry>
+                <mesh filename="package://rosbot_description/meshes/rosbot/wheel_b.dae"/>
+            </geometry>
+            <origin xyz="0 0 0" rpy="0 0 0"/>
+        </visual>
+    </link>
+    <joint name="wheel_right_forward_joint" type="fixed">
+        <parent link="base_link"/>
+        <child link="wheel_right_forward_link"/>
+        <origin xyz="${wheel_separation_x/2} -${wheel_separation_y/2} 0.015" rpy="0 0 0"/>
+    </joint>
 </robot>

Commit message: make the wheels continuous

File: rosbot_description/urdf/rosbot.urdf.xacro (robot description, xacro)
@@ -11,4 +11,7 @@
             </geometry>
             <origin xyz="0 0 0" rpy="${pi/2} 0 ${pi/2}"/>
+            <material name="orange">
+                <color rgba="0.4 0.4 0.4 1"/>
+            </material>
         </visual>
     </link>
@@ -24,4 +27,7 @@
             </geometry>
             <origin xyz="0 0 0.015" rpy="${pi/2} 0 ${pi/2}"/>
+            <material name="grey">
+                <color rgba="1 0.27 0 1"/>
+            </material>
         </visual>
     </link>
@@ -39,8 +45,9 @@
         </visual>
     </link>
-    <joint name="wheel_left_back_joint" type="fixed">
+    <joint name="wheel_left_back_joint" type="continuous">
         <parent link="base_link"/>
         <child link="wheel_left_back_link"/>
         <origin xyz="-${wheel_separation_x/2} ${wheel_separation_y/2} 0.015" rpy="0 0 0"/>
+        <axis xyz="0 1 0"/>
     </joint>
     <link name="wheel_left_forward_link">
@@ -52,8 +59,9 @@
         </visual>
     </link>
-    <joint name="wheel_left_forward_joint" type="fixed">
+    <joint name="wheel_left_forward_joint" type="continuous">
         <parent link="base_link"/>
         <child link="wheel_left_forward_link"/>
         <origin xyz="${wheel_separation_x/2} ${wheel_separation_y/2} 0.015" rpy="0 0 0"/>
+        <axis xyz="0 1 0"/>
     </joint>
     <link name="wheel_right_back_link">
@@ -65,8 +73,9 @@
         </visual>
     </link>
-    <joint name="wheel_right_back_joint" type="fixed">
+    <joint name="wheel_right_back_joint" type="continuous">
         <parent link="base_link"/>
         <child link="wheel_right_back_link"/>
         <origin xyz="-${wheel_separation_x/2} -${wheel_separation_y/2} 0.015" rpy="0 0 0"/>
+        <axis xyz="0 1 0"/>
     </joint>
     <link name="wheel_right_forward_link">
@@ -78,8 +87,9 @@
         </visual>
     </link>
-    <joint name="wheel_right_forward_joint" type="fixed">
+    <joint name="wheel_right_forward_joint" type="continuous">
         <parent link="base_link"/>
         <child link="wheel_right_forward_link"/>
         <origin xyz="${wheel_separation_x/2} -${wheel_separation_y/2} 0.015" rpy="0 0 0"/>
+        <axis xyz="0 1 0"/>
     </joint>
 </robot>

Commit message: add collision and inertial of base link

File: rosbot_description/urdf/rosbot.urdf.xacro (robot description, xacro)
@@ -15,4 +15,17 @@
             </material>
         </visual>
+        <collision>
+            <geometry>
+                <box size="0.197 0.150 0.080"/>
+            </geometry>
+            <origin xyz=" 0 0 0.038" rpy="0 0 0"/>
+        </collision>
+        <inertial>
+            <mass value="1.728" />
+            <inertia ixx="0.004162" ixy="0.0"     ixz="0.0"
+                                    iyy="0.00651" iyz="0.0"
+                                                  izz="0.008828" />
+            <origin xyz="0.0 0.0 0.038" rpy="0.0 0.0 0.0" />
+          </inertial>
     </link>
     <joint name="base_joint" type="fixed">

Commit message: add collision for wheels

File: rosbot_description/urdf/rosbot.urdf.xacro (robot description, xacro)
@@ -2,4 +2,5 @@
 <robot name="rosbot" xmlns:xacro="http://ros.org/wiki/xacro">
     <xacro:property name="wheel_radius" value="0.0425"/>
+    <xacro:property name="wheel_thickness" value="0.0455"/>
     <xacro:property name="wheel_separation_x" value="0.106"/>
     <xacro:property name="wheel_separation_y" value="0.192"/>
@@ -57,4 +58,10 @@
             <origin xyz="0 0 0" rpy="0 0 0"/>
         </visual>
+        <collision>
+            <geometry>
+                <cylinder radius="${wheel_radius}" length="${wheel_thickness}"/>
+            </geometry>
+            <origin xyz="0 0 0" rpy="${pi/2} 0 0"/>
+        </collision>
     </link>
     <joint name="wheel_left_back_joint" type="continuous">
@@ -71,4 +78,10 @@
             <origin xyz="0 0 0" rpy="0 0 0"/>
         </visual>
+        <collision>
+            <geometry>
+                <cylinder radius="${wheel_radius}" length="${wheel_thickness}"/>
+            </geometry>
+            <origin xyz="0 0 0" rpy="${pi/2} 0 0"/>
+        </collision>
     </link>
     <joint name="wheel_left_forward_joint" type="continuous">
@@ -85,4 +98,10 @@
             <origin xyz="0 0 0" rpy="0 0 0"/>
         </visual>
+        <collision>
+            <geometry>
+                <cylinder radius="${wheel_radius}" length="${wheel_thickness}"/>
+            </geometry>
+            <origin xyz="0 0 0" rpy="${pi/2} 0 0"/>
+        </collision>
     </link>
     <joint name="wheel_right_back_joint" type="continuous">
@@ -99,4 +118,10 @@
             <origin xyz="0 0 0" rpy="0 0 0"/>
         </visual>
+        <collision>
+            <geometry>
+                <cylinder radius="${wheel_radius}" length="${wheel_thickness}"/>
+            </geometry>
+            <origin xyz="0 0 0" rpy="${pi/2} 0 0"/>
+        </collision>
     </link>
     <joint name="wheel_right_forward_joint" type="continuous">

Commit message: add inertial of wheels

File: rosbot_description/urdf/rosbot.urdf.xacro (robot description, xacro)
@@ -2,5 +2,5 @@
 <robot name="rosbot" xmlns:xacro="http://ros.org/wiki/xacro">
     <xacro:property name="wheel_radius" value="0.0425"/>
-    <xacro:property name="wheel_thickness" value="0.0455"/>
+    <xacro:property name="wheel_thickness" value="0.036"/>
     <xacro:property name="wheel_separation_x" value="0.106"/>
     <xacro:property name="wheel_separation_y" value="0.192"/>
@@ -28,5 +28,5 @@
                                                   izz="0.008828" />
             <origin xyz="0.0 0.0 0.038" rpy="0.0 0.0 0.0" />
-          </inertial>
+        </inertial>
     </link>
     <joint name="base_joint" type="fixed">
@@ -64,4 +64,10 @@
             <origin xyz="0 0 0" rpy="${pi/2} 0 0"/>
         </collision>
+        <inertial>
+            <mass value="0.074" />
+            <inertia ixx="0.000041" ixy="0.0"    ixz="0.0"
+                                  iyy="0.000067" iyz="0.0"
+                                               izz="0.000041" />
+        </inertial>
     </link>
     <joint name="wheel_left_back_joint" type="continuous">
@@ -84,4 +90,10 @@
             <origin xyz="0 0 0" rpy="${pi/2} 0 0"/>
         </collision>
+        <inertial>
+            <mass value="0.074" />
+            <inertia ixx="0.000041" ixy="0.0"    ixz="0.0"
+                                  iyy="0.000067" iyz="0.0"
+                                               izz="0.000041" />
+        </inertial>
     </link>
     <joint name="wheel_left_forward_joint" type="continuous">
@@ -104,4 +116,10 @@
             <origin xyz="0 0 0" rpy="${pi/2} 0 0"/>
         </collision>
+        <inertial>
+            <mass value="0.074" />
+            <inertia ixx="0.000041" ixy="0.0"    ixz="0.0"
+                                  iyy="0.000067" iyz="0.0"
+                                               izz="0.000041" />
+        </inertial>
     </link>
     <joint name="wheel_right_back_joint" type="continuous">
@@ -124,4 +142,10 @@
             <origin xyz="0 0 0" rpy="${pi/2} 0 0"/>
         </collision>
+        <inertial>
+            <mass value="0.074" />
+            <inertia ixx="0.000041" ixy="0.0"    ixz="0.0"
+                                  iyy="0.000067" iyz="0.0"
+                                               izz="0.000041" />
+        </inertial>
     </link>
     <joint name="wheel_right_forward_joint" type="continuous">

Commit message: add imu link

File: rosbot_description/urdf/rosbot.urdf.xacro (robot description, xacro)
@@ -157,3 +157,9 @@
         <axis xyz="0 1 0"/>
     </joint>
+    <link name="imu_link"/>
+    <joint name="imu_joint" type="fixed">
+        <parent link="base_link"/>
+        <child link="imu_link"/>
+        <origin xyz="0.003 -0.0495 0.04332" rpy="0.0 0.0 0.0" />
+    </joint>
 </robot>

Commit message: add laser scan link to urdf

File: rosbot_description/urdf/rosbot.urdf.xacro (robot description, xacro)
@@ -14,5 +14,5 @@
             </geometry>
             <origin xyz="0 0 0" rpy="${pi/2} 0 ${pi/2}"/>
-            <material name="orange">
+            <material name="grey">
                 <color rgba="0.4 0.4 0.4 1"/>
             </material>
@@ -43,5 +43,5 @@
             </geometry>
             <origin xyz="0 0 0.015" rpy="${pi/2} 0 ${pi/2}"/>
-            <material name="grey">
+            <material name="orange">
                 <color rgba="1 0.27 0 1"/>
             </material>
@@ -163,3 +163,32 @@
         <origin xyz="0.003 -0.0495 0.04332" rpy="0.0 0.0 0.0" />
     </joint>
+    <link name="laser_link">
+        <visual>
+            <geometry>
+                <mesh filename="package://rosbot_description/meshes/rosbot/laser_link.STL" scale="0.55 0.55 0.55"/>
+            </geometry>
+            <origin xyz="0 0 0" rpy="0 0 ${pi}"/>
+            <material name="black">
+                <color rgba="0.1 0.1 0.1 1"/>
+            </material>
+        </visual>
+        <collision>
+            <geometry>
+                <mesh filename="package://rosbot_description/meshes/rosbot/laser_link.STL" scale="0.55 0.55 0.55"/>
+            </geometry>
+            <origin xyz="0 0 0" rpy="0 0 ${pi}"/>
+        </collision>
+        <inertial>
+            <origin xyz="-0.011945780406062 -0.000381929217680526 -0.0170649378129477" rpy="0 0 0" />
+            <mass value="0.073084435549317" />
+            <inertia ixx="1.96074931730795E-05" ixy="-3.62091076640009E-07" ixz="4.28230084046735E-07"
+                     iyy="2.40983835136327E-05" iyz="1.50180909250652E-08"
+                     izz="4.14184164228595E-05" />
+        </inertial>
+    </link>
+    <joint name="laser_joint" type="fixed">
+        <parent link="base_link"/>
+        <child link="laser_link"/>
+        <origin xyz="-0.045 0 0.165" rpy="0 0 0"/>
+    </joint>
 </robot>
